Commit message: Vehicle V2: puff-port shutters; cross-team requests in AGENTS.md
- Four sliding puff-port shutters (Blender links, prismatic joints,
  JointPositionControllers). AirCushion opens them in proportion to the
  vent force, so Gazebo/RViz/Foxglove show which vents fire. Visual only,
  inside the 1.5 m footprint. New render puff_port_open.png.
- AGENTS.md: open requests to Person 1 (obstacle inflation 1.7 m for V2;
  LiDAR transform needs no change) and Person 2 (hover energy 0.0133 %/m,
  hover hold drain, V2 track figures). Mode-selection text updated to the
  hover-first policy. CLAUDE.md imports AGENTS.md for Claude Code agents.
- Plugin changes still need a Gazebo build and the v2_* tests.

Co-Authored-By: Claude Opus 5.5 <noreply@anthropic.com>

File: autonomous_tidal_vehicle_ws/src/tidal_vehicle_description/urdf/hovercraft_v2.urdf (robot description, URDF)
Before this commit: robot hovercraft_v2, 13 links, 12 joints
Links:
- added link puff_bow_left, mass 0.5; collision box size=0.26 0.006 0.14; visual mesh filename=package://tidal_vehicle_description/models/hovercraft_v2/me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
- added link puff_bow_right, mass 0.5; collision box size=0.26 0.006 0.14; visual mesh filename=package://tidal_vehicle_description/models/hovercraft_v2/me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
- added link puff_stern_left, mass 0.5; collision box size=0.26 0.006 0.14; visual mesh filename=package://tidal_vehicle_description/models/hovercraft_v2/me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
- added link puff_stern_right, mass 0.5; collision box size=0.26 0.006 0.14; visual mesh filename=package://tidal_vehicle_description/models/hovercraft_v2/me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
- link base_link: mass 147.8 -> 145.8
Joints:
- added joint puff_bow_left_joint: type prismatic, parent base_link, child puff_bow_left, origin xyz=0.74 0.7 0.01 rpy=0 0 0, axis -1 0 0, limit lower=-0.02 upper=0.28 effort=20 velocity=1.0
- added joint puff_bow_right_joint: type prismatic, parent base_link, child puff_bow_right, origin xyz=0.74 -0.7 0.01 rpy=0 0 0, axis -1 0 0, limit lower=-0.02 upper=0.28 effort=20 velocity=1.0
- added joint puff_stern_left_joint: type prismatic, parent base_link, child puff_stern_left, origin xyz=-0.74 0.7 0.01 rpy=0 0 0, axis 1 0 0, limit lower=-0.02 upper=0.28 effort=20 velocity=1.0
- added joint puff_stern_right_joint: type prismatic, parent base_link, child puff_stern_right, origin xyz=-0.74 -0.7 0.01 rpy=0 0 0, axis 1 0 0, limit lower=-0.02 upper=0.28 effort=20 velocity=1.0
