Commit message: Person 4: V3 front LiDAR, mangrove visual fix, track hysteresis, optional IMU/slope features
- Mangroves: move each visible mesh onto its collision proxy. The GLB trunk is
  off its origin, so trees were drawn 8-18 m from their proxies and the GPU
  LiDAR reported "phantom trees" on free cells (e.g. mangrove_18 at (74.4, 0.2)).
  Notice to Person 3 in AGENTS.md (item 19).
- Version 3: front near-field LiDAR on the bow bay (/points_front, 180 deg,
  -25..+5 deg, 0.2-15 m), Blender model, SDF/URDF and bridge; not yet merged
  into /scan.
- lidar_scan_node: keep Person 1's corridor-profile ground filter as the active
  one; add Person 4's map-free slope filter levelled by the IMU as an option
  (slope_ground_filter_deg, level_with_imu; off by default).
- vehicle_mobility_node: TRACK exits only after the climb stays low (hysteresis,
  V2 10 deg / V3 4 deg); optional command ramps, IMU attitude, downhill speed
  cap and track braking on steep descents (all off by default).
- Clean Ctrl+C shutdown in Person 4 nodes; executable flags on new V3 scripts.
- Version 3 heavy-load presentation variant (Blender, visual only).

Tests: simulation 41, autonomy 50, safety 20, operator 10 pass; V2 integration
mission completes (delivery + return, 79 s).

Co-Authored-By: Claude Opus 5.5 <noreply@anthropic.com>

File: autonomous_tidal_vehicle_ws/src/tidal_vehicle_description/urdf/hovercraft_v3.urdf (robot description, URDF)
Before this commit: robot hovercraft_v3, 20 links, 19 joints
Links:
- added link lidar_front_link
Joints:
- added joint lidar_front_link_joint: type fixed, parent base_link, child lidar_front_link, origin xyz=1.18 0 0.54 rpy=0 0 0
